Commit message: Provisional implement the model of T-frog

File: t_frog_description/urdf/t_frog.xacro (robot description, xacro)
@@ -4,11 +4,6 @@
   <!-- Constants for robot dimensions -->
   <xacro:property name="PI" value="3.1415926535897931"/>
-  <xacro:property name="width" value="0.1" /> <!-- Square dimensions (widthxwidth) of beams -->
-  <xacro:property name="height1" value="2" /> <!-- Link 1 -->
-  <xacro:property name="height2" value="1" /> <!-- Link 2 -->
-  <xacro:property name="height3" value="1" /> <!-- Link 3 -->
   <xacro:property name="camera_link" value="0.05"/> <!-- Size of square 'camera' box -->
   <xacro:property name="hokuyo_link" value="0.1" /> <!-- Size of square 'hokuyo' box -->
-  <xacro:property name="axel_offset" value="0.05"/> <!-- Space btw top of beam and the each joint -->
   <!-- Import all Gazebo-customization elements, including Gazebo colors -->
   <xacro:include filename="$(find t_frog_description)/urdf/t_frog.gazebo" />
@@ -26,20 +21,20 @@
   <link name="base_link">
     <collision>
-      <origin xyz="0 0 .1" rpy="0 0 0"/>
-      <geometry>
-	<box size=".4 .2 .1"/>
-      </geometry>
-    </collision>
-    <visual>
-      <origin xyz="0 0 .1" rpy="0 0 0"/>
-      <geometry>
-	<box size=".4 .2 .1"/>
+      <origin xyz="0 0 0.1" rpy="0 0 0"/>
+      <geometry>
+	<box size=".3 .2 .1"/>
+      </geometry>
+    </collision>
+    <visual>
+      <origin xyz="0 0 0.1" rpy="0 0 0"/>
+      <geometry>
+	<box size=".3 .2 .1"/>
       </geometry>
       <material name="orange"/>
     </visual>
     <collision>
-      <origin xyz="-0.15 0 0.03" rpy="0 0 0"/>
-      <geometry>
-	<sphere radius="0.02"/>
+      <origin xyz="0.15 0 0.05" rpy="0 0 0"/>
+      <geometry>
+	<sphere radius="0.028"/>
       </geometry>
       <surface>
@@ -55,14 +50,37 @@
     </collision>
     <visual>
-      <origin xyz="-0.15 0 0.03" rpy="0 0 0"/>
-      <geometry>
-	<sphere radius="0.02"/>
+      <origin xyz="0.15 0 0.05" rpy="0 0 0"/>
+      <geometry>
+	<sphere radius="0.028"/>
       </geometry>
       <material name="orange"/>
     </visual>
-    <inertial>
-       <mass value="1e-5" />
-       <origin xyz="0 0 .1 " rpy="0 0 0"/>
-       <inertia ixx="1e-6" ixy="0" ixz="0" iyy="1e-6" iyz="0" izz="1e-6" />
+    <collision>
+      <origin xyz="-0.15 0 0.05" rpy="0 0 0"/>
+      <geometry>
+	<sphere radius="0.028"/>
+      </geometry>
+      <surface>
+        <friction>
+          <ode>
+	    <mu>0</mu>
+	    <mu2>0</mu2>
+	    <slip1>1.0</slip1>
+	    <slip2>1.0</slip2>
+	  </ode>
+        </friction>
+      </surface>
+    </collision>
+    <visual>
+      <origin xyz="-0.15 0 0.05" rpy="0 0 0"/>
+      <geometry>
+	<sphere radius="0.028"/>
+      </geometry>
+      <material name="orange"/>
+    </visual>
+    <inertial>
+       <mass value="5" />
+       <origin xyz="0 0 0.1" rpy="0 0 0"/>
+       <inertia ixx="5" ixy="0" ixz="0" iyy="5" iyz="0" izz="5" />
     </inertial>
   </link>
@@ -81,11 +99,11 @@
     </visual>
     <inertial>
-      <mass value="1e-5" />
+      <mass value="0.1" />
       <origin xyz="0 0.03 0"/>
-      <inertia ixx="1e-6" ixy="0" ixz="0" iyy="1e-6" iyz="0" izz="1e-6" />
+      <inertia ixx="0.1" ixy="0" ixz="0" iyy="0.1" iyz="0" izz="0.1" />
     </inertial>
   </link>
   <joint type="revolute" name="left_wheel_hinge">
-    <origin xyz="0.1 0.13 0.1" rpy="0 0 0"/>
+    <origin xyz="0 0.13 0.12" rpy="0 0 0"/>
     <child link="left_wheel">left_wheel</child>
     <parent link="base_link">base_link</parent>
@@ -107,11 +125,11 @@
     </visual>
     <inertial>
-      <mass value="1e-5" />
+      <mass value="0.1" />
       <origin xyz="0 -0.03 0"/>
-      <inertia ixx="1e-6" ixy="0" ixz="0" iyy="1e-6" iyz="0" izz="1e-6" />
+      <inertia ixx="0.1" ixy="0" ixz="0" iyy="0.1" iyz="0" izz="0.1" />
     </inertial>
   </link>
   <joint type="revolute" name="right_wheel_hinge">
-    <origin xyz="0.1 -0.13 0.1" rpy="0 0 0"/>
+    <origin xyz="0 -0.13 0.12" rpy="0 0 0"/>
     <child link="right_wheel">right_wheel</child>
     <parent link="base_link">base_link</parent>
@@ -121,5 +139,5 @@
   <joint name="hokuyo_joint" type="fixed">
     <axis xyz="0 1 0"/>
-    <origin xyz="0 0 0.175" rpy="0 0 0"/>
+    <origin xyz="0.15 0 0.175" rpy="0 0 0"/>
     <parent link="base_link"/>
     <child link="hokuyo_link"/>
@@ -139,12 +157,12 @@
     </visual>
     <inertial>
-      <mass value="1e-5"/>
-      <origin xyz="0 0 0" rpy="0 0 0"/>
-      <inertia ixx="1e-6" ixy="0" ixz="0" iyy="1e-6" iyz="0" izz="1e-6"/>
+      <mass value="1"/>
+      <origin xyz="0 0 0" rpy="0 0 0"/>
+      <inertia ixx="1" ixy="0" ixz="0" iyy="1" iyz="0" izz="1"/>
     </inertial>
   </link>
   <joint name="camera_joint" type="fixed">
     <axis xyz="0 1 0" />
-    <origin xyz="0.2 0 0.175" rpy="0 0 0"/>
+    <origin xyz="-0.15 0 0.175" rpy="0 0 0"/>
     <parent link="base_link"/>
     <child link="camera_link"/>
@@ -165,7 +183,7 @@
     </visual>
     <inertial>
-      <mass value="1e-5" />
-      <origin xyz="0 0 0" rpy="0 0 0"/>
-      <inertia ixx="1e-6" ixy="0" ixz="0" iyy="1e-6" iyz="0" izz="1e-6" />
+      <mass value="1"/>
+      <origin xyz="0 0 0" rpy="0 0 0"/>
+      <inertia ixx="1" ixy="0" ixz="0" iyy="1" iyz="0" izz="1"/>
     </inertial>
   </link>

Commit message: Change the controller type

File: t_frog_description/urdf/t_frog.xacro (robot description, xacro)
@@ -11,11 +11,9 @@
   <xacro:include filename="$(find t_frog_description)/urdf/materials.xacro" />
   <!-- Used for fixing robot to Gazebo 'base_link' -->
-  <!--
-  <link name="world"/>
+  <!--link name="world"/>
   <joint name="continuous" type="continuous">
     <parent link="world"/>
     <child link="base_link"/>
-  </joint>
-  -->
+  </joint-->
   <!-- Base Link -->
   <link name="base_link">
